Commit message: 0.0.7

File: urdf/arm_b.xacro (robot description, xacro)
@@ -6,4 +6,8 @@
 							origin_rpy = "0 0 0"
 							origin_xyz = "0 0 0"
+							mass="1024"
+              				ixx="170.667" ixy="0" ixz="0"
+              				iyy="170.667" iyz="0"
+              				izz="170.667"
 							size = "1 1 1" />
 	<xacro:m_joint 			name = "${l00}_${l01}"
@@ -17,4 +21,8 @@
     						origin_rpy = "0 0 0"
     						origin_xyz = "0 0 0.2"
+    						mass="57.906"
+              				ixx="12.679" ixy="0" ixz="0"
+              				iyy="12.679" iyz="0"
+              				izz="0.651"
     						radius = "0.35"
     						length="0.4" />
@@ -29,4 +37,8 @@
     						origin_rpy = "0 0 0"
     						origin_xyz = "0 0 0.5"
+    						mass="57.906"
+              				ixx="12.679" ixy="0" ixz="0"
+              				iyy="12.679" iyz="0"
+              				izz="0.651"
     						radius = "0.10"
     						length="1" />
@@ -41,4 +53,8 @@
 							origin_rpy = "0 0 0"
 							origin_xyz = "0 0 0.5"
+							mass="57.906"
+              				ixx="12.679" ixy="0" ixz="0"
+             		 		iyy="12.679" iyz="0"
+              				izz="0.651"
 							radius = "0.10"
 							length="1" />
@@ -53,4 +69,8 @@
 							origin_rpy = "0 0 0"
 							origin_xyz = "0 0 0.5"
+							mass="57.906"
+              				ixx="12.679" ixy="0" ixz="0"
+              				iyy="12.679" iyz="0"
+              				izz="0.651"
 							radius = "0.10"
 							length="1" />
@@ -65,4 +85,8 @@
 							origin_rpy = "0 0 0"
 							origin_xyz = "0 0 0.1"
+							mass="18.056"
+              				ixx="0.479" ixy="0" ixz="0"
+              				iyy="0.479" iyz="0"
+              				izz="0.204"
 							radius = "0.2"
 							length="0.2" />

File: urdf/link_joint.xacro (robot description, xacro)
@@ -10,6 +10,17 @@
     	</joint>
     </xacro:macro>
-	<xacro:macro name="m_link_cylinder" params="name origin_xyz origin_rpy radius length">
+	<xacro:macro name="m_link_cylinder" params="name origin_xyz origin_rpy radius length mass ixx ixy ixz iyy iyz izz">
     <link name="${name}">
+      <inertial>
+        <mass value="${mass}" />
+        <origin rpy="${origin_rpy}" xyz="${origin_xyz}" />
+        <inertia ixx="${ixx}" ixy="${ixy}" ixz="${ixz}" iyy="${iyy}" iyz="${iyz}" izz="${izz}" />
+      </inertial>
+      <collision>
+        <origin rpy="${origin_rpy}" xyz="${origin_xyz}" />
+        <geometry>
+          <cylinder radius="${radius}" length="${length}" />
+        </geometry>
+      </collision>
       <visual>
         <origin rpy="${origin_rpy}" xyz="${origin_xyz}" />
@@ -20,6 +31,17 @@
     </link>
   </xacro:macro>
-  <xacro:macro name="m_link_box" params="name origin_xyz origin_rpy size">
+  <xacro:macro name="m_link_box" params="name origin_xyz origin_rpy size mass ixx ixy ixz iyy iyz izz">
     <link name="${name}">
+      <inertial>
+        <mass value="${mass}" />
+        <origin rpy="${origin_rpy}" xyz="${origin_xyz}" />
+        <inertia ixx="${ixx}" ixy="${ixy}" ixz="${ixz}" iyy="${iyy}" iyz="${iyz}" izz="${izz}" />
+      </inertial>
+      <collision>
+        <origin rpy="${origin_rpy}" xyz="${origin_xyz}" />
+        <geometry>
+          <box size="${size}" />
+        </geometry>
+      </collision>
       <visual>
         <origin rpy="${origin_rpy}" xyz="${origin_xyz}" />

Commit message: 0.0.9

File: urdf/arm_b.xacro (robot description, xacro)
@@ -18,4 +18,14 @@
 							parent = "${l00}"
 							child = "${l01}" />
+	<transmission name="trans_${l00}_${l01}">
+      <type>transmission_interface/SimpleTransmission</type>
+      <joint name="${l00}_${l01}">
+        <hardwareInterface>hardware_interface/EffortJointInterface</hardwareInterface>
+      </joint>
+      <actuator name="motor_${l00}_${l01}">
+        <hardwareInterface>hardware_interface/EffortJointInterface</hardwareInterface>
+        <mechanicalReduction>1</mechanicalReduction>
+      </actuator>
+    </transmission>
     <xacro:m_link_cylinder 	name = "${l01}"
     						origin_rpy = "0 0 0"
@@ -34,4 +44,14 @@
     						parent = "${l01}"
     						child = "${l02}" />
+    <transmission name="trans_${l01}_${l02}">
+      <type>transmission_interface/SimpleTransmission</type>
+      <joint name="${l01}_${l02}">
+        <hardwareInterface>hardware_interface/EffortJointInterface</hardwareInterface>
+      </joint>
+      <actuator name="motor_${l00}_${l01}">
+        <hardwareInterface>hardware_interface/EffortJointInterface</hardwareInterface>
+        <mechanicalReduction>1</mechanicalReduction>
+      </actuator>
+    </transmission>
     <xacro:m_link_cylinder 	name = "${l02}"
     						origin_rpy = "0 0 0"
@@ -43,5 +63,5 @@
     						radius = "0.10"
     						length="1" />
-    <xacro:m_joint 			name = "${l02}_${l03}"
+    <!-- <xacro:m_joint 			name = "${l02}_${l03}"
     						type = "revolute"
     						axis_xyz = "0 1 0"
@@ -91,3 +111,7 @@
 							radius = "0.2"
 							length="0.2" />
+ -->
+ <gazebo>
+ 	<plugin name = "gazebo_ros_control" filename = "libgazebo_ros_control.so" />
+ </gazebo>
 </robot>

Commit message: 0.0.10

File: urdf/arm_b.xacro (robot description, xacro)
@@ -17,21 +17,12 @@
 							origin_xyz = "0 0 0.5"
 							parent = "${l00}"
-							child = "${l01}" />
-	<transmission name="trans_${l00}_${l01}">
-      <type>transmission_interface/SimpleTransmission</type>
-      <joint name="${l00}_${l01}">
-        <hardwareInterface>hardware_interface/EffortJointInterface</hardwareInterface>
-      </joint>
-      <actuator name="motor_${l00}_${l01}">
-        <hardwareInterface>hardware_interface/EffortJointInterface</hardwareInterface>
-        <mechanicalReduction>1</mechanicalReduction>
-      </actuator>
-    </transmission>
+							child = "${l01}"
+							limit_e="1000" limit_l="-3.14" limit_u="3.14" limit_v="0.5"/>
     <xacro:m_link_cylinder 	name = "${l01}"
     						origin_rpy = "0 0 0"
     						origin_xyz = "0 0 0.2"
-    						mass="57.906"
-              				ixx="12.679" ixy="0" ixz="0"
-              				iyy="12.679" iyz="0"
+    						mass="10"
+              				ixx="1" ixy="0" ixz="0"
+              				iyy="1" iyz="0"
               				izz="0.651"
     						radius = "0.35"
@@ -43,25 +34,16 @@
     						origin_xyz = "0 0 0.4"
     						parent = "${l01}"
-    						child = "${l02}" />
-    <transmission name="trans_${l01}_${l02}">
-      <type>transmission_interface/SimpleTransmission</type>
-      <joint name="${l01}_${l02}">
-        <hardwareInterface>hardware_interface/EffortJointInterface</hardwareInterface>
-      </joint>
-      <actuator name="motor_${l00}_${l01}">
-        <hardwareInterface>hardware_interface/EffortJointInterface</hardwareInterface>
-        <mechanicalReduction>1</mechanicalReduction>
-      </actuator>
-    </transmission>
+    						child = "${l02}"
+    						limit_e="1000" limit_l="-0.75" limit_u="0.75" limit_v="0.5"/>
     <xacro:m_link_cylinder 	name = "${l02}"
     						origin_rpy = "0 0 0"
     						origin_xyz = "0 0 0.5"
-    						mass="57.906"
-              				ixx="12.679" ixy="0" ixz="0"
-              				iyy="12.679" iyz="0"
+    						mass="12.906"
+              				ixx="1" ixy="0" ixz="0"
+              				iyy="1.679" iyz="0"
               				izz="0.651"
     						radius = "0.10"
     						length="1" />
-    <!-- <xacro:m_joint 			name = "${l02}_${l03}"
+    <xacro:m_joint 			name = "${l02}_${l03}"
     						type = "revolute"
     						axis_xyz = "0 1 0"
@@ -69,11 +51,12 @@
     						origin_xyz = "0 0 1"
     						parent = "${l02}"
-    						child = "${l03}" />
+    						child = "${l03}"
+    						limit_e="1000" limit_l="-0.75" limit_u="1.5" limit_v="0.5"/>
 	<xacro:m_link_cylinder 	name = "${l03}"
 							origin_rpy = "0 0 0"
 							origin_xyz = "0 0 0.5"
-							mass="57.906"
-              				ixx="12.679" ixy="0" ixz="0"
-             		 		iyy="12.679" iyz="0"
+							mass="12.906"
+              				ixx="1.679" ixy="0" ixz="0"
+             		 		iyy="1.679" iyz="0"
               				izz="0.651"
 							radius = "0.10"
@@ -85,11 +68,12 @@
     						origin_xyz = "0 0 1"
     						parent = "${l03}"
-    						child = "${l04}" />
+    						child = "${l04}"
+    						limit_e="1000" limit_l="0" limit_u="2.5" limit_v="0.5"/>
 	<xacro:m_link_cylinder 	name = "${l04}"
 							origin_rpy = "0 0 0"
 							origin_xyz = "0 0 0.5"
-							mass="57.906"
-              				ixx="12.679" ixy="0" ixz="0"
-              				iyy="12.679" iyz="0"
+							mass="12.906"
+              				ixx="1.679" ixy="0" ixz="0"
+              				iyy="1.679" iyz="0"
               				izz="0.651"
 							radius = "0.10"
@@ -101,15 +85,15 @@
     						origin_xyz = "0 0 1"
     						parent = "${l04}"
-    						child = "${l05}" />
+    						child = "${l05}"
+    						limit_e="1000" limit_l="-3.14" limit_u="3.14" limit_v="0.5"/>
 	<xacro:m_link_cylinder 	name = "${l05}"
 							origin_rpy = "0 0 0"
 							origin_xyz = "0 0 0.1"
-							mass="18.056"
-              				ixx="0.479" ixy="0" ixz="0"
-              				iyy="0.479" iyz="0"
+							mass="2.056"
+              				ixx="0.179" ixy="0" ixz="0"
+              				iyy="0.179" iyz="0"
               				izz="0.204"
 							radius = "0.2"
 							length="0.2" />
- -->
  <gazebo>
  	<plugin name = "gazebo_ros_control" filename = "libgazebo_ros_control.so" />

File: urdf/link_joint.xacro (robot description, xacro)
@@ -1,13 +1,23 @@
 <?xml version='1.0' ?>
 <robot name = "arm" xmlns:xacro="http://www.ros.org/wiki/xacro">
-	<xacro:macro name = "m_joint" params = "name type axis_xyz origin_rpy origin_xyz parent child">
+	<xacro:macro name = "m_joint" params = "name type axis_xyz origin_rpy origin_xyz parent child limit_e limit_l limit_u limit_v">
 		<joint name="${name}" type="${type}">
 	      <axis xyz="${axis_xyz}" />
-	      <limit effort="1000.0" lower="-3.14" upper = "3.14" velocity = "0.5"/>
+	      <limit effort="${limit_e}" lower="${limit_l}" upper="${limit_u}" velocity="${limit_v}" />
 	      <origin rpy="${origin_rpy}" xyz="${origin_xyz}" />
 	      <parent link="${parent}" />
 	      <child link="${child}" />
     	</joint>
-    </xacro:macro>
+      <transmission name="trans_${name}">
+      <type>transmission_interface/SimpleTransmission</type>
+      <joint name="${name}">
+        <hardwareInterface>hardware_interface/EffortJointInterface</hardwareInterface>
+      </joint>
+      <actuator name="motor_${name}">
+        <hardwareInterface>hardware_interface/EffortJointInterface</hardwareInterface>
+        <mechanicalReduction>1</mechanicalReduction>
+      </actuator>
+    </transmission>
+  </xacro:macro>
 	<xacro:macro name="m_link_cylinder" params="name origin_xyz origin_rpy radius length mass ixx ixy ixz iyy iyz izz">
     <link name="${name}">

Commit message: 0.0.11

File: urdf/arm_b.xacro (robot description, xacro)
@@ -19,5 +19,13 @@
 							child = "${l01}"
 							limit_e="1000" limit_l="-3.14" limit_u="3.14" limit_v="0.5"/>
-    <xacro:m_link_cylinder 	name = "${l01}"
+	<xacro:m_link_mesh name="${l01}"
+              origin_rpy="0 0 0" origin_xyz="0 0 -0.1"
+              mass="157.633"
+              ixx="13.235" ixy="0" ixz="0"
+              iyy="13.235" iyz="0"
+              izz="9.655"
+              meshfile="package://arm_a/meshes/Link1-v2.stl"
+              meshscale="0.001 0.001 0.001" />
+    <!-- <xacro:m_link_cylinder 	name = "${l01}"
     						origin_rpy = "0 0 0"
     						origin_xyz = "0 0 0.2"
@@ -27,6 +35,6 @@
               				izz="0.651"
     						radius = "0.35"
-    						length="0.4" />
-    <xacro:m_joint 			name = "${l01}_${l02}"
+    						length="0.4" /> -->
+    <!-- <xacro:m_joint 			name = "${l01}_${l02}"
     						type = "revolute"
     						axis_xyz = "0 1 0"
@@ -95,5 +103,5 @@
               				izz="0.204"
 							radius = "0.2"
-							length="0.2" />
+							length="0.2" /> -->
  <gazebo>
  	<plugin name = "gazebo_ros_control" filename = "libgazebo_ros_control.so" />

File: urdf/link_joint.xacro (robot description, xacro)
@@ -62,3 +62,25 @@
     </link>
   </xacro:macro>
+  <xacro:macro name="m_link_mesh" params="name origin_xyz origin_rpy meshfile meshscale mass ixx ixy ixz iyy iyz izz">
+    <link name="${name}">
+      <inertial>
+        <mass value="${mass}" />
+        <origin rpy="${origin_rpy}" xyz="${origin_xyz}" />
+        <inertia ixx="${ixx}" ixy="${ixy}" ixz="${ixz}" iyy="${iyy}" iyz="${iyz}" izz="${izz}" />
+      </inertial>
+      <collision>
+        <origin rpy="${origin_rpy}" xyz="${origin_xyz}" />
+        <geometry>
+          <mesh filename="${meshfile}" scale="${meshscale}"/>
+        </geometry>
+      </collision>
+      <visual>
+        <origin rpy="${origin_rpy}" xyz="${origin_xyz}" />
+        <geometry>
+          <mesh filename="${meshfile}" scale="${meshscale}"/>
+        </geometry>
+        <material name="light_black"/>
+      </visual>
+    </link>
+  </xacro:macro>
 </robot>

Commit message: 1.0.2

File: urdf/arm_b.xacro (robot description, xacro)
@@ -19,13 +19,5 @@
 							child = "${l01}"
 							limit_e="1000" limit_l="-3.14" limit_u="3.14" limit_v="0.5"/>
-	<xacro:m_link_mesh name="${l01}"
-              origin_rpy="0 0 0" origin_xyz="0 0 -0.1"
-              mass="157.633"
-              ixx="13.235" ixy="0" ixz="0"
-              iyy="13.235" iyz="0"
-              izz="9.655"
-              meshfile="package://arm_a/meshes/Link1-v2.stl"
-              meshscale="0.001 0.001 0.001" />
-    <!-- <xacro:m_link_cylinder 	name = "${l01}"
+    <xacro:m_link_cylinder 	name = "${l01}"
     						origin_rpy = "0 0 0"
     						origin_xyz = "0 0 0.2"
@@ -35,6 +27,6 @@
               				izz="0.651"
     						radius = "0.35"
-    						length="0.4" /> -->
-    <!-- <xacro:m_joint 			name = "${l01}_${l02}"
+    						length="0.4" />
+    <xacro:m_joint 			name = "${l01}_${l02}"
     						type = "revolute"
     						axis_xyz = "0 1 0"
@@ -103,5 +95,5 @@
               				izz="0.204"
 							radius = "0.2"
-							length="0.2" /> -->
+							length="0.2" />
  <gazebo>
  	<plugin name = "gazebo_ros_control" filename = "libgazebo_ros_control.so" />

File: urdf/arm_c.xacro (robot description, xacro)
@@ -3,4 +3,5 @@
 	<xacro:include filename = "$(find arm_a)/urdf/link_joint.xacro" />
 	<xacro:include filename = "$(find arm_a)/urdf/robot_parameters.xacro" />
+	<xacro:include filename = "$(find realsense2_description)/urdf/_d435.urdf.xacro" />
 	<xacro:m_link_box 		name = "${l00}"
 							origin_rpy = "0 0 0"
@@ -17,11 +18,12 @@
 							origin_xyz = "0 0 0.5"
 							parent = "${l00}"
-							child = "${l01}" />
+							child = "${l01}"
+							limit_e="1000" limit_l="-3.14" limit_u="3.14" limit_v="0.5"/>
     <xacro:m_link_cylinder 	name = "${l01}"
     						origin_rpy = "0 0 0"
     						origin_xyz = "0 0 0.2"
-    						mass="57.906"
-              				ixx="12.679" ixy="0" ixz="0"
-              				iyy="12.679" iyz="0"
+    						mass="10"
+              				ixx="1" ixy="0" ixz="0"
+              				iyy="1" iyz="0"
               				izz="0.651"
     						radius = "0.35"
@@ -33,13 +35,84 @@
     						origin_xyz = "0 0 0.4"
     						parent = "${l01}"
-    						child = "${l02}" />
+    						child = "${l02}"
+    						limit_e="1000" limit_l="-0.75" limit_u="0.75" limit_v="0.5"/>
     <xacro:m_link_cylinder 	name = "${l02}"
     						origin_rpy = "0 0 0"
     						origin_xyz = "0 0 0.5"
-    						mass="57.906"
-              				ixx="12.679" ixy="0" ixz="0"
-              				iyy="12.679" iyz="0"
+    						mass="12.906"
+              				ixx="1" ixy="0" ixz="0"
+              				iyy="1.679" iyz="0"
               				izz="0.651"
     						radius = "0.10"
     						length="1" />
+    <xacro:m_joint 			name = "${l02}_${l03}"
+    						type = "revolute"
+    						axis_xyz = "0 1 0"
+    						origin_rpy = "0 0 0"
+    						origin_xyz = "0 0 1"
+    						parent = "${l02}"
+    						child = "${l03}"
+    						limit_e="1000" limit_l="-0.75" limit_u="1.5" limit_v="0.5"/>
+	<xacro:m_link_cylinder 	name = "${l03}"
+							origin_rpy = "0 0 0"
+							origin_xyz = "0 0 0.5"
+							mass="12.906"
+              				ixx="1.679" ixy="0" ixz="0"
+             		 		iyy="1.679" iyz="0"
+              				izz="0.651"
+							radius = "0.10"
+							length="1" />
+    <xacro:m_joint 			name = "${l03}_${l04}"
+    						type = "revolute"
+    						axis_xyz = "0 1 0"
+    						origin_rpy = "0 0 0"
+    						origin_xyz = "0 0 1"
+    						parent = "${l03}"
+    						child = "${l04}"
+    						limit_e="1000" limit_l="0" limit_u="2.5" limit_v="0.5"/>
+	<xacro:m_link_cylinder 	name = "${l04}"
+							origin_rpy = "0 0 0"
+							origin_xyz = "0 0 0.5"
+							mass="12.906"
+              				ixx="1.679" ixy="0" ixz="0"
+              				iyy="1.679" iyz="0"
+              				izz="0.651"
+							radius = "0.10"
+							length="1" />
+    <joint name="${l04}_${l05}" type="fixed">
+	    <parent link="${l04}"/>
+	    <child link="${l05}"/>
+	    <origin xyz="0 0 1"/>
+  	</joint>
+	<xacro:m_link_box 		name = "${l05}"
+							origin_rpy = "0 0 0"
+							origin_xyz = "0 0 0.05"
+							mass="10"
+              				ixx="0.1" ixy="0" ixz="0"
+              				iyy="0.1" iyz="0"
+              				izz="0.05"
+							size = "0.4 0.4 0.1" />
+    <xacro:m_joint 			name = "${l05}_${l06}"
+    						type = "revolute"
+    						axis_xyz = "0 0 1"
+    						origin_rpy = "0 0 0"
+    						origin_xyz = "0 0 0.1"
+    						parent = "${l05}"
+    						child = "${l06}"
+    						limit_e="1000" limit_l="-3.14" limit_u="3.14" limit_v="0.5"/>
+	<xacro:m_link_cylinder 	name = "${l06}"
+							origin_rpy = "0 0 0"
+							origin_xyz = "0 0 0.05"
+							mass="2.056"
+              				ixx="0.179" ixy="0" ixz="0"
+              				iyy="0.179" iyz="0"
+              				izz="0.204"
+							radius = "0.15"
+							length="0.1" />
+	<xacro:sensor_d435 name="camera" topics_ns="camera" parent="${l05}" publish_pointcloud="true">
+    <origin xyz="-0.2 0 0.1" rpy="0 -1.57 0" />
+  </xacro:sensor_d435>
+ <gazebo>
+ 	<plugin name = "gazebo_ros_control" filename = "libgazebo_ros_control.so" />
+ </gazebo>
 </robot>

File: urdf/link_joint.xacro (robot description, xacro)
@@ -84,3 +84,25 @@
     </link>
   </xacro:macro>
+  <!-- Testing Depth Camera -->
+  <xacro:macro name = "m_link_camera" params="name origin_xyz origin_rpy size mass ixx ixy ixz iyy iyz izz">
+    <link name="${name}">
+      <inertial>
+        <mass value="${mass}" />
+        <origin rpy="${origin_rpy}" xyz="${origin_xyz}" />
+        <inertia ixx="${ixx}" ixy="${ixy}" ixz="${ixz}" iyy="${iyy}" iyz="${iyz}" izz="${izz}" />
+      </inertial>
+      <collision>
+        <origin rpy="${origin_rpy}" xyz="${origin_xyz}" />
+        <geometry>
+          <box size="${size}" />
+        </geometry>
+      </collision>
+      <visual>
+        <origin rpy="${origin_rpy}" xyz="${origin_xyz}" />
+        <geometry>
+          <box size="${size}" />
+        </geometry>
+      </visual>
+    </link>
+  </xacro:macro>
 </robot>

File: urdf/robot_parameters.xacro (robot description, xacro)
@@ -7,3 +7,5 @@
   <xacro:property name="l04" value="link_4" />
   <xacro:property name="l05" value="link_5" />
+  <xacro:property name="l06" value="link_6" />
+  <xacro:property name="l07" value="link_7" />
 </robot>
